Commit message: Added distance sensors

File: description/lidar.xacro (robot description, xacro)
@@ -11,5 +11,5 @@
                 <cylinder radius="0.05" length="0.04"/>
             </geometry>
-            <material name="red"/>
+            <material name="blue"/>
         </visual>
         <collision>
@@ -23,6 +23,6 @@
     </link>
     <gazebo reference="laser_frame">
-        <material>Gazebo/Red</material>
-        <sensor name="laser" type="gpu_ray">
+        <material>Gazebo/Blue</material>
+        <sensor name="lidar" type="gpu_ray">
             <pose> 0 0 0 0 0 0 </pose>
             <visualize>true</visualize>
@@ -41,5 +41,5 @@
                 </range>
             </ray>
-            <plugin name="gazebo_ros_head_hokuyo_controller" filename="libgazebo_ros_gpu_laser.so">
+            <plugin name="gazebo_lidar" filename="libgazebo_ros_gpu_laser.so">
                 <topicName>/scan</topicName>
                 <frameName>laser_frame</frameName>

Commit message: Updated Models

File: description/lidar.xacro (robot description, xacro)
@@ -1,8 +1,32 @@
 <?xml version="1.0"?>
 <robot xmlns:xacro="http://www.ros.org/wiki/xacro" >
+    <joint name="laser_arm_joint" type="fixed">
+        <parent link="chassis"/>
+        <child link="laser_arm"/>
+        <origin xyz=".90 0 0.25" rpy="0 0 0"/>
+    </joint>
+    <link name="laser_arm">
+        <visual>
+            <geometry>
+                <box size=".2 .2 0.1"/>
+            </geometry>
+            <material name="white"/>
+        </visual>
+        <collision>
+            <geometry>
+                <box size=".2 .2 0.1"/>
+            </geometry>
+        </collision>
+        <xacro:inertial_box mass="2" x=".2" y=".2" z=".1">
+            <origin xyz="0 0 0" rpy="0 0 0"/>
+        </xacro:inertial_box>
+    </link>
+    <gazebo reference="laser_arm">
+        <material>Gazebo/White</material>
+    </gazebo>
     <joint name="laser_joint" type="fixed">
-        <parent link="chassis"/>
+        <parent link="laser_arm"/>
         <child link="laser_frame"/>
-        <origin xyz=".90 0 0.25" rpy="0 0 0"/>
+        <origin xyz=".05 0 -.07" rpy="0 0 0"/>
     </joint>
     <link name="laser_frame">
