Commit message: Spring break

File: description/distance_sensors.xacro (robot description, xacro)
@@ -5,5 +5,5 @@
         <parent link="chassis"/>
         <child link="distance_sensor_left"/>
-        <origin xyz=".9 -.3 .5" rpy="0 0.20943632679 0"/>
+        <origin xyz=".85 -.25 .37" rpy="0 0.20943632679 0"/>
     </joint>
     <link name="distance_sensor_left">
@@ -52,5 +52,5 @@
         <parent link="chassis"/>
         <child link="distance_sensor_right"/>
-        <origin xyz=".9 .3 .5" rpy="0 0.20943632679 0"/>
+        <origin xyz=".85 .25 .37" rpy="0 0.20943632679 0"/>
     </joint>
     <link name="distance_sensor_right">

File: description/gazebo_control.xacro (robot description, xacro)
@@ -2,42 +2,24 @@
 <robot xmlns:xacro="http://www.ros.org/wiki/xacro">
     <gazebo>
-        <plugin name="skid_steer_drive_controller" filename="libgazebo_ros_skid_steer_drive.so">
+        <plugin name="diff_drive" filename="libgazebo_ros_diff_drive.so">
+            <leftJoint>right_drive_wheel_1_joint</leftJoint>
+            <rightJoint>left_drive_wheel_1_joint</rightJoint>
+            <wheelSeparation>.5</wheelSeparation>
+            <wheelDiameter>0.2</wheelDiameter>
+            <wheelTorque>200</wheelTorque>
+            <wheelAcceleration>10.0</wheelAcceleration>
             <updateRate>100.0</updateRate>
-            <robotNamespace>/</robotNamespace>
-            <leftFrontJoint>left_drive_wheel_3_joint</leftFrontJoint>
-            <rightFrontJoint>right_drive_wheel_3_joint</rightFrontJoint>
-            <leftRearJoint>left_drive_wheel_1_joint</leftRearJoint>
-            <rightRearJoint>right_drive_wheel_1_joint</rightRearJoint>
-            <wheelSeparation>1.0</wheelSeparation>
-            <wheelDiameter>0.3</wheelDiameter>
-            <torque>200</torque>
-            <wheelAcceleration>10.0</wheelAcceleration>
             <commandTopic>cmd_vel</commandTopic>
             <odometryTopic>odom</odometryTopic>
-            <robotBaseFrame>base_link</robotBaseFrame>
             <odometryFrame>odom</odometryFrame>
-            <covariance_x>0.0001</covariance_x>
-            <covariance_y>0.0001</covariance_y>
-            <covariance_yaw>0.01</covariance_yaw>
-            <!--publish_odom>true</publish_odom>
-            <publishOdomTF>true</publishOdomTF-->
-            <publishWheelTF>true</publishWheelTF>
-            <broadcastTF>true</broadcastTF>
-        </plugin>
-        <!--plugin name="diff_drive" filename="libgazebo_ros_diff_drive.so">
-            <leftJoint>left_drive_wheel_3_joint</leftJoint>
-            <rightJoint>right_drive_wheel_3_joint</rightJoint>
-            <wheelSeparation>1.0</wheelSeparation>
-            <wheelDiameter>0.3</wheelDiameter>
-            <wheelTorque>200</wheelTorque>
-            <wheelAcceleration>10.0</wheelAcceleration>
-            <commandTopic>cmd_vel</commandTopic>
-            <odometryTopic>odom</odometryTopic>
+            <odometrySource>1</odometrySource>
             <robotBaseFrame>base_link</robotBaseFrame>
             <publish_odom>true</publish_odom>
             <publishOdomTF>true</publishOdomTF>
             <publishWheelTF>true</publishWheelTF>
+            <publishTf>1</publishTf>
+            <publishWheelJointState>true</publishWheelJointState>
             <rosDebugLevel>na</rosDebugLevel>
-        </plugin-->
+        </plugin>
     </gazebo>
 </robot>

File: description/lidar.xacro (robot description, xacro)
@@ -4,5 +4,5 @@
         <parent link="chassis"/>
         <child link="laser_arm"/>
-        <origin xyz=".90 0 0.25" rpy="0 0 0"/>
+        <origin xyz=".90 0 0.2" rpy="0 0 0"/>
     </joint>
     <link name="laser_arm">

File: description/rover_core.xacro (robot description, xacro)
@@ -25,22 +25,22 @@
         <parent link="base_link"/>
         <child link="chassis"/>
-        <origin xyz="-0.1 0 0"/>
+        <origin xyz="-0.1 0 0.1"/>
     </joint>
     <link name="chassis">
         <visual>
-            <origin xyz=".5 0 .25"/>
+            <origin xyz=".5 0 .2"/>
             <geometry>
-                <box size=".75 .6 0.5"/>
+                <box size=".75 .5 0.35"/>
             </geometry>
             <material name="white"/>
         </visual>
         <collision>
-            <origin xyz=".5 0 .25"/>
+            <origin xyz=".5 0 .2"/>
             <geometry>
-                <box size=".75 .6 0.5"/>
+                <box size=".75 .5 0.35"/>
             </geometry>
         </collision>
         <xacro:inertial_box mass="42" x="1" y="1" z=".5">
-            <origin xyz=".5 0 .25" rpy="0 0 0"/>
+            <origin xyz=".5 0 .2" rpy="0 0 0"/>
         </xacro:inertial_box>
     </link>
@@ -52,5 +52,5 @@
         <parent link="base_link"/>
         <child link="left_drive_wheel_1_train"/>
-        <origin xyz=".15 -.3 0" rpy="${pi/2} 0 0"/>
+        <origin xyz=".25 -.25 0.1" rpy="-${pi/2} 0 0"/>
         <axis xyz="0 0 1"/>
     </joint>
@@ -58,5 +58,5 @@
         <visual>
             <geometry>
-                <cylinder radius=".15" length=".2"/>
+                <cylinder radius=".1" length=".08"/>
             </geometry>
             <material name="black"/>
@@ -64,8 +64,8 @@
         <collision>
             <geometry>
-                <cylinder radius=".15" length=".2"/>
+                <cylinder radius=".1" length=".08"/>
             </geometry>
         </collision>
-        <xacro:inertial_cylinder mass="3" length=".2" radius=".15">
+        <xacro:inertial_cylinder mass="3" length=".08" radius=".1">
             <origin xyz="0 0 0" rpy="0 0 0"/>
         </xacro:inertial_cylinder>
@@ -74,8 +74,9 @@
         <material>Gazebo/Black</material>
     </gazebo>
-    <joint name="left_drive_wheel_3_joint" type="continuous">
+    <!-- LEFT DRIVE WHEEL 3 LINK -->
+    <joint name="left_drive_wheel_3_joint" type="fixed">
         <parent link="base_link"/>
         <child link="left_drive_wheel_3_train"/>
-        <origin xyz=".6 -.3 0" rpy="${pi/2} 0 0"/>
+        <origin xyz=".6 -.25 0.1" rpy="-${pi/2} 0 0"/>
         <axis xyz="0 0 1"/>
     </joint>
@@ -83,5 +84,5 @@
         <visual>
             <geometry>
-                <cylinder radius=".15" length=".2"/>
+                <cylinder radius=".1" length=".08"/>
             </geometry>
             <material name="black"/>
@@ -89,8 +90,8 @@
         <collision>
             <geometry>
-                <cylinder radius=".15" length=".2"/>
+                <cylinder radius=".1" length=".08"/>
             </geometry>
         </collision>
-        <xacro:inertial_cylinder mass="3" length=".2" radius=".15">
+        <xacro:inertial_cylinder mass="3" length=".08" radius=".1">
             <origin xyz="0 0 0" rpy="0 0 0"/>
         </xacro:inertial_cylinder>
@@ -98,4 +99,6 @@
     <gazebo reference="left_drive_wheel_3_train">
         <material>Gazebo/Black</material>
+        <mu1 value="0.001"/>
+        <mu2 value="0.001"/>
     </gazebo>
     <!-- RIGHT DRIVE WHEEL 1 LINK -->
@@ -103,5 +106,5 @@
         <parent link="base_link"/>
         <child link="right_drive_wheel_1_train"/>
-        <origin xyz=".15 .3 0" rpy="-${pi/2} 0 0"/>
+        <origin xyz=".25 .25 0.1" rpy="${pi/2} 0 0"/>
         <axis xyz="0 0 -1"/>
     </joint>
@@ -109,5 +112,5 @@
         <visual>
             <geometry>
-                <cylinder radius=".15" length=".2"/>
+                <cylinder radius=".1" length=".08"/>
             </geometry>
             <material name="black"/>
@@ -115,8 +118,8 @@
         <collision>
             <geometry>
-                <cylinder radius=".15" length=".2"/>
+                <cylinder radius=".1" length=".08"/>
             </geometry>
         </collision>
-        <xacro:inertial_cylinder mass="3" length=".2" radius=".15">
+        <xacro:inertial_cylinder mass="3" length=".08" radius=".1">
             <origin xyz="0 0 0" rpy="0 0 0"/>
         </xacro:inertial_cylinder>
@@ -126,8 +129,8 @@
     </gazebo>
     <!-- RIGHT DRIVE WHEEL 3 LINK -->
-    <joint name="right_drive_wheel_3_joint" type="continuous">
+    <joint name="right_drive_wheel_3_joint" type="fixed">
         <parent link="base_link"/>
         <child link="right_drive_wheel_3_train"/>
-        <origin xyz=".6 .3 0" rpy="-${pi/2} 0 0"/>
+        <origin xyz=".6 .25 0.1" rpy="${pi/2} 0 0"/>
         <axis xyz="0 0 -1"/>
     </joint>
@@ -135,5 +138,5 @@
         <visual>
             <geometry>
-                <cylinder radius=".15" length=".2"/>
+                <cylinder radius=".1" length=".08"/>
             </geometry>
             <material name="black"/>
@@ -141,8 +144,8 @@
         <collision>
             <geometry>
-                <cylinder radius=".15" length=".2"/>
+                <cylinder radius=".1" length=".08"/>
             </geometry>
         </collision>
-        <xacro:inertial_cylinder mass="3" length=".2" radius=".15">
+        <xacro:inertial_cylinder mass="3" length=".08" radius=".1">
             <origin xyz="0 0 0" rpy="0 0 0"/>
         </xacro:inertial_cylinder>
@@ -150,4 +153,6 @@
     <gazebo reference="right_drive_wheel_3_train">
         <material>Gazebo/Black</material>
+        <mu1 value="0.001"/>
+        <mu2 value="0.001"/>
     </gazebo>
 </robot>
